Commit message: improve file paths for meshes.

File: piper_description/urdf/piper_description.urdf (robot description, URDF)
Before this commit: robot piper, 11 links, 10 joints
Links:
- removed link dummy_link
- link link6: mass 0.007 -> 0.00699089613564366
Joints:
- removed joint base_to_dummy
- joint joint1: limit lower=-2.618 upper=2.618 effort=100 velocity=5 -> lower=-2.618 upper=2.168 effort=100 velocity=5

File: piper_description/urdf/piper_description.xacro (robot description, xacro)
@@ -4,25 +4,16 @@
   xmlns:xacro="http://ros.org/wiki/xacro">
 <!-- world -->
-  <!-- <link name="world"/>
+  <link name="world"/>
   <joint name="fixed_base_joint" type="fixed">
       <parent link="world"/>
       <child link="base_link"/>
-  </joint> -->
-<!-- piper -->
+  </joint>
+<!-- arm -->
 <link
-    name="arm_base">
-    <inertial>
-      <origin
-        xyz="-0.00473641164191482 2.56829134630247E-05 0.041451518036016"
-        rpy="0 0 0" />
-      <mass
-        value="1.02" />
-      <inertia
-        ixx="0.00267433"
-        ixy="-0.00000073"
-        ixz="-0.00017389"
-        iyy="0.00282612"
-        iyz="0.0000004"
-        izz="0.00089624" />
+    name="base_link">
+    <inertial>
+            <origin xyz="-0.00473641164191482 2.56829134630247E-05 0.041451518036016" rpy="0 0 0" />
+            <mass value="1.02" />
+            <inertia ixx="0.00267433" ixy="-0.00000073" ixz="-0.00017389" iyy="0.00282612" iyz="0.0000004" izz="0.00089624" />
     </inertial>
     <visual>
@@ -53,16 +44,7 @@
     name="link1">
     <inertial>
-      <origin
-        xyz="0.000121504734057468 0.000104632162460536 -0.00438597309559853"
-        rpy="0 0 0" />
-      <mass
-        value="0.71" />
-      <inertia
-        ixx="0.00048916"
-        ixy="-0.00000036"
-        ixz="-0.00000224"
-        iyy="0.00040472"
-        iyz="-0.00000242"
-        izz="0.00043982" />
+            <origin xyz="0.000121504734057468 0.000104632162460536 -0.00438597309559853" rpy="0 0 0" />
+            <mass value="0.71" />
+            <inertia ixx="0.00048916" ixy="-0.00000036" ixz="-0.00000224" iyy="0.00040472" iyz="-0.00000242" izz="0.00043982" />
     </inertial>
     <visual>
@@ -97,5 +79,5 @@
       rpy="0 0 0" />
     <parent
-      link="arm_base" />
+      link="base_link" />
     <child
       link="link1" />
@@ -111,16 +93,7 @@
     name="link2">
     <inertial>
-      <origin
-        xyz="0.198666145229743 -0.010926924140076 0.00142121714502687"
-        rpy="0 0 0" />
-      <mass
-        value="1.17" />
-      <inertia
-        ixx="0.00116918"
-        ixy="-0.00180037"
-        ixz="0.00025146"
-        iyy="0.06785384"
-        iyz="-0.00000455"
-        izz="0.06774489" />
+            <origin xyz="0.198666145229743 -0.010926924140076 0.00142121714502687" rpy="0 0 0" />
+            <mass value="1.17" />
+            <inertia ixx="0.00116918" ixy="-0.00180037" ixz="0.00025146" iyy="0.06785384" iyz="-0.00000455" izz="0.06774489" />
     </inertial>
     <visual>
@@ -170,16 +143,7 @@
     name="link3">
     <inertial>
-      <origin
-        xyz="-0.0202737662122021 -0.133914995944595 -0.000458682652737356"
-        rpy="0 0 0" />
-      <mass
-        value="0.5" />
-      <inertia
-        ixx="0.01361711"
-        ixy="0.00165794"
-        ixz="-0.00000048"
-        iyy="0.00045024"
-        iyz="-0.00000045"
-        izz="0.01380322" />
+            <origin xyz="-0.0202737662122021 -0.133914995944595 -0.000458682652737356" rpy="0 0 0" />
+            <mass value="0.5" />
+            <inertia ixx="0.01361711" ixy="0.00165794" ixz="-0.00000048" iyy="0.00045024" iyz="-0.00000045" izz="0.01380322" />
     </inertial>
     <visual>
@@ -229,16 +193,7 @@
     name="link4">
     <inertial>
-      <origin
-        xyz="-9.66635791618542E-05 0.000876064475651083 -0.00496880904640868"
-        rpy="0 0 0" />
-      <mass
-        value="0.38" />
-      <inertia
-        ixx="0.00018501"
-        ixy="0.00000054"
-        ixz="0.00000120"
-        iyy="0.00018965"
-        iyz="-0.00000841"
-        izz="0.00015484" />
+            <origin xyz="-9.66635791618542E-05 0.000876064475651083 -0.00496880904640868" rpy="0 0 0" />
+            <mass value="0.38" />
+            <inertia ixx="0.00018501" ixy="0.00000054" ixz="0.00000120" iyy="0.00018965" iyz="-0.00000841" izz="0.00015484" />
     </inertial>
     <visual>
@@ -287,16 +242,7 @@
     name="link5">
     <inertial>
-      <origin
-        xyz="-4.10554118924211E-05 -0.0566486692356075 -0.0037205791677906"
-        rpy="0 0 0" />
-      <mass
-        value="0.383" />
-      <inertia
-        ixx="0.00166169"
-        ixy="0.00000006"
-        ixz="-0.00000007"
-        iyy="0.00018510"
-        iyz="0.00001026"
-        izz="0.00164321" />
+            <origin xyz="-4.10554118924211E-05 -0.0566486692356075 -0.0037205791677906" rpy="0 0 0" />
+            <mass value="0.383" />
+            <inertia ixx="0.00166169" ixy="0.00000006" ixz="-0.00000007" iyy="0.00018510" iyz="0.00001026" izz="0.00164321" />
     </inertial>
     <visual>
@@ -345,16 +291,7 @@
     name="link6">
     <inertial>
-      <origin
-        xyz="-8.82590762930069E-05 9.0598378529832E-06 -0.002"
-        rpy="0 0 0" />
-      <mass
-        value="0.007" />
-      <inertia
-        ixx="5.73015540542155E-07"
-        ixy="-1.98305403089247E-22"
-        ixz="-7.2791893904596E-23"
-        iyy="5.73015540542155E-07"
-        iyz="-3.4146026640245E-24"
-        izz="1.06738869138926E-06" />
+            <origin xyz="-8.82590762930069E-05 9.0598378529832E-06 -0.002" rpy="0 0 0" />
+            <mass value="0.00699089613564366" />
+            <inertia ixx="5.73015540542155E-07" ixy="-1.98305403089247E-22" ixz="-7.2791893904596E-23" iyy="5.73015540542155E-07" iyz="-3.4146026640245E-24" izz="1.06738869138926E-06" />
     </inertial>
     <visual>
@@ -463,5 +400,5 @@
         ixy="-0.00000113"
         ixz="0.00000021"
-        iyy="0.00000781"
+        iyy="-0.00000113"
         iyz="-0.00001372"
         izz="0.0000747" />
@@ -521,5 +458,5 @@
         ixy="-0.00000113"
         ixz="0.00000021"
-        iyy="0.00000781"
+        iyy="-0.00000113"
         iyz="-0.00001372"
         izz="0.0000747" />
@@ -590,6 +527,7 @@
 <!-- gazebo -->
   <gazebo>
-    <plugin name="gazebo_ros_control" filename="libgazebo_ros_control.so">
+    <plugin name="gazebo_ros2_control" filename="libgazebo_ros2_control.so">
         <robotNamespace>/piper</robotNamespace>
+        <parameters> $(find piper_gazebo)/config/ros2_controllers.yaml </parameters>
         <legacyModeNS>true</legacyModeNS>
     </plugin>

File: piper_description/urdf/piper_description_gazebo.xacro (robot description, xacro)
@@ -1,5 +1,5 @@
 <?xml version="1.0" encoding="utf-8"?>
 <robot
-  name="gazebo"
+  name="piper"
   xmlns:xacro="http://ros.org/wiki/xacro">
 <!-- world -->
@@ -9,42 +9,33 @@
       <child link="base_link"/>
   </joint>
-<!-- gazebo -->
+<!-- arm -->
 <link
     name="base_link">
     <inertial>
-      <origin
-        xyz="-0.00473641164191482 2.56829134630247E-05 0.041451518036016"
-        rpy="0 0 0" />
-      <mass
-        value="1.02" />
-      <inertia
-        ixx="0.00267433"
-        ixy="-0.00000073"
-        ixz="-0.00017389"
-        iyy="0.00282612"
-        iyz="0.0000004"
-        izz="0.00089624" />
-    </inertial>
-    <visual>
-      <origin
-        xyz="0 0 0"
-        rpy="0 0 0" />
-      <geometry>
-        <mesh
-          filename="package://piper_description/meshes/base_link.STL" />
-      </geometry>
-      <material
-        name="">
-        <color
-          rgba="0.792156862745098 0.819607843137255 0.933333333333333 1" />
-      </material>
-    </visual>
-    <collision>
-      <origin
-        xyz="0 0 0"
-        rpy="0 0 0" />
-      <geometry>
-        <mesh
-          filename="package://piper_description/meshes/base_link.STL" />
+            <origin xyz="-0.00473641164191482 2.56829134630247E-05 0.041451518036016" rpy="0 0 0" />
+            <mass value="1.02" />
+            <inertia ixx="0.00267433" ixy="-0.00000073" ixz="-0.00017389" iyy="0.00282612" iyz="0.0000004" izz="0.00089624" />
+    </inertial>
+    <visual>
+      <origin
+        xyz="0 0 0"
+        rpy="0 0 0" />
+      <geometry>
+        <mesh
+          filename="file://$(find piper_description)/meshes/base_link.STL" />
+      </geometry>
+      <material
+        name="">
+        <color
+          rgba="0.792156862745098 0.819607843137255 0.933333333333333 1" />
+      </material>
+    </visual>
+    <collision>
+      <origin
+        xyz="0 0 0"
+        rpy="0 0 0" />
+      <geometry>
+        <mesh
+          filename="file://$(find piper_description)/meshes/base_link.STL" />
       </geometry>
     </collision>
@@ -53,38 +44,29 @@
     name="link1">
     <inertial>
-      <origin
-        xyz="0.000121504734057468 0.000104632162460536 -0.00438597309559853"
-        rpy="0 0 0" />
-      <mass
-        value="0.71" />
-      <inertia
-        ixx="0.00048916"
-        ixy="-0.00000036"
-        ixz="-0.00000224"
-        iyy="0.00040472"
-        iyz="-0.00000242"
-        izz="0.00043982" />
-    </inertial>
-    <visual>
-      <origin
-        xyz="0 0 0"
-        rpy="0 0 0" />
-      <geometry>
-        <mesh
-          filename="package://piper_description/meshes/link1.STL" />
-      </geometry>
-      <material
-        name="">
-        <color
-          rgba="0.792156862745098 0.819607843137255 0.933333333333333 1" />
-      </material>
-    </visual>
-    <collision>
-      <origin
-        xyz="0 0 0"
-        rpy="0 0 0" />
-      <geometry>
-        <mesh
-          filename="package://piper_description/meshes/link1.STL" />
+            <origin xyz="0.000121504734057468 0.000104632162460536 -0.00438597309559853" rpy="0 0 0" />
+            <mass value="0.71" />
+            <inertia ixx="0.00048916" ixy="-0.00000036" ixz="-0.00000224" iyy="0.00040472" iyz="-0.00000242" izz="0.00043982" />
+    </inertial>
+    <visual>
+      <origin
+        xyz="0 0 0"
+        rpy="0 0 0" />
+      <geometry>
+        <mesh
+          filename="file://$(find piper_description)/meshes/link1.STL" />
+      </geometry>
+      <material
+        name="">
+        <color
+          rgba="0.792156862745098 0.819607843137255 0.933333333333333 1" />
+      </material>
+    </visual>
+    <collision>
+      <origin
+        xyz="0 0 0"
+        rpy="0 0 0" />
+      <geometry>
+        <mesh
+          filename="file://$(find piper_description)/meshes/link1.STL" />
       </geometry>
     </collision>
@@ -111,38 +93,29 @@
     name="link2">
     <inertial>
-      <origin
-        xyz="0.198666145229743 -0.010926924140076 0.00142121714502687"
-        rpy="0 0 0" />
-      <mass
-        value="1.17" />
-      <inertia
-        ixx="0.00116918"
-        ixy="-0.00180037"
-        ixz="0.00025146"
-        iyy="0.06785384"
-        iyz="-0.00000455"
-        izz="0.06774489" />
-    </inertial>
-    <visual>
-      <origin
-        xyz="0 0 0"
-        rpy="0 0 0" />
-      <geometry>
-        <mesh
-          filename="package://piper_description/meshes/link2.STL" />
-      </geometry>
-      <material
-        name="">
-        <color
-          rgba="0.792156862745098 0.819607843137255 0.933333333333333 1" />
-      </material>
-    </visual>
-    <collision>
-      <origin
-        xyz="0 0 0"
-        rpy="0 0 0" />
-      <geometry>
-        <mesh
-          filename="package://piper_description/meshes/link2.STL" />
+            <origin xyz="0.198666145229743 -0.010926924140076 0.00142121714502687" rpy="0 0 0" />
+            <mass value="1.17" />
+            <inertia ixx="0.00116918" ixy="-0.00180037" ixz="0.00025146" iyy="0.06785384" iyz="-0.00000455" izz="0.06774489" />
+    </inertial>
+    <visual>
+      <origin
+        xyz="0 0 0"
+        rpy="0 0 0" />
+      <geometry>
+        <mesh
+          filename="file://$(find piper_description)/meshes/link2.STL" />
+      </geometry>
+      <material
+        name="">
+        <color
+          rgba="0.792156862745098 0.819607843137255 0.933333333333333 1" />
+      </material>
+    </visual>
+    <collision>
+      <origin
+        xyz="0 0 0"
+        rpy="0 0 0" />
+      <geometry>
+        <mesh
+          filename="file://$(find piper_description)/meshes/link2.STL" />
       </geometry>
     </collision>
@@ -170,38 +143,29 @@
     name="link3">
     <inertial>
-      <origin
-        xyz="-0.0202737662122021 -0.133914995944595 -0.000458682652737356"
-        rpy="0 0 0" />
-      <mass
-        value="0.5" />
-      <inertia
-        ixx="0.01361711"
-        ixy="0.00165794"
-        ixz="-0.00000048"
-        iyy="0.00045024"
-        iyz="-0.00000045"
-        izz="0.01380322" />
-    </inertial>
-    <visual>
-      <origin
-        xyz="0 0 0"
-        rpy="0 0 0" />
-      <geometry>
-        <mesh
-          filename="package://piper_description/meshes/link3.STL" />
-      </geometry>
-      <material
-        name="">
-        <color
-          rgba="0.792156862745098 0.819607843137255 0.933333333333333 1" />
-      </material>
-    </visual>
-    <collision>
-      <origin
-        xyz="0 0 0"
-        rpy="0 0 0" />
-      <geometry>
-        <mesh
-          filename="package://piper_description/meshes/link3.STL" />
+            <origin xyz="-0.0202737662122021 -0.133914995944595 -0.000458682652737356" rpy="0 0 0" />
+            <mass value="0.5" />
+            <inertia ixx="0.01361711" ixy="0.00165794" ixz="-0.00000048" iyy="0.00045024" iyz="-0.00000045" izz="0.01380322" />
+    </inertial>
+    <visual>
+      <origin
+        xyz="0 0 0"
+        rpy="0 0 0" />
+      <geometry>
+        <mesh
+          filename="file://$(find piper_description)/meshes/link3.STL" />
+      </geometry>
+      <material
+        name="">
+        <color
+          rgba="0.792156862745098 0.819607843137255 0.933333333333333 1" />
+      </material>
+    </visual>
+    <collision>
+      <origin
+        xyz="0 0 0"
+        rpy="0 0 0" />
+      <geometry>
+        <mesh
+          filename="file://$(find piper_description)/meshes/link3.STL" />
       </geometry>
     </collision>
@@ -229,38 +193,29 @@
     name="link4">
     <inertial>
-      <origin
-        xyz="-9.66635791618542E-05 0.000876064475651083 -0.00496880904640868"
-        rpy="0 0 0" />
-      <mass
-        value="0.38" />
-      <inertia
-        ixx="0.00018501"
-        ixy="0.00000054"
-        ixz="0.00000120"
-        iyy="0.00018965"
-        iyz="-0.00000841"
-        izz="0.00015484" />
-    </inertial>
-    <visual>
-      <origin
-        xyz="0 0 0"
-        rpy="0 0 0" />
-      <geometry>
-        <mesh
-          filename="package://piper_description/meshes/link4.STL" />
-      </geometry>
-      <material
-        name="">
-        <color
-          rgba="0.792156862745098 0.819607843137255 0.933333333333333 1" />
-      </material>
-    </visual>
-    <collision>
-      <origin
-        xyz="0 0 0"
-        rpy="0 0 0" />
-      <geometry>
-        <mesh
-          filename="package://piper_description/meshes/link4.STL" />
+            <origin xyz="-9.66635791618542E-05 0.000876064475651083 -0.00496880904640868" rpy="0 0 0" />
+            <mass value="0.38" />
+            <inertia ixx="0.00018501" ixy="0.00000054" ixz="0.00000120" iyy="0.00018965" iyz="-0.00000841" izz="0.00015484" />
+    </inertial>
+    <visual>
+      <origin
+        xyz="0 0 0"
+        rpy="0 0 0" />
+      <geometry>
+        <mesh
+          filename="file://$(find piper_description)/meshes/link4.STL" />
+      </geometry>
+      <material
+        name="">
+        <color
+          rgba="0.792156862745098 0.819607843137255 0.933333333333333 1" />
+      </material>
+    </visual>
+    <collision>
+      <origin
+        xyz="0 0 0"
+        rpy="0 0 0" />
+      <geometry>
+        <mesh
+          filename="file://$(find piper_description)/meshes/link4.STL" />
       </geometry>
     </collision>
@@ -287,38 +242,29 @@
     name="link5">
     <inertial>
-      <origin
-        xyz="-4.10554118924211E-05 -0.0566486692356075 -0.0037205791677906"
-        rpy="0 0 0" />
-      <mass
-        value="0.383" />
-      <inertia
-        ixx="0.00166169"
-        ixy="0.00000006"
-        ixz="-0.00000007"
-        iyy="0.00018510"
-        iyz="0.00001026"
-        izz="0.00164321" />
-    </inertial>
-    <visual>
-      <origin
-        xyz="0 0 0"
-        rpy="0 0 0" />
-      <geometry>
-        <mesh
-          filename="package://piper_description/meshes/link5.STL" />
-      </geometry>
-      <material
-        name="">
-        <color
-          rgba="0.792156862745098 0.819607843137255 0.933333333333333 1" />
-      </material>
-    </visual>
-    <collision>
-      <origin
-        xyz="0 0 0"
-        rpy="0 0 0" />
-      <geometry>
-        <mesh
-          filename="package://piper_description/meshes/link5.STL" />
+            <origin xyz="-4.10554118924211E-05 -0.0566486692356075 -0.0037205791677906" rpy="0 0 0" />
+            <mass value="0.383" />
+            <inertia ixx="0.00166169" ixy="0.00000006" ixz="-0.00000007" iyy="0.00018510" iyz="0.00001026" izz="0.00164321" />
+    </inertial>
+    <visual>
+      <origin
+        xyz="0 0 0"
+        rpy="0 0 0" />
+      <geometry>
+        <mesh
+          filename="file://$(find piper_description)/meshes/link5.STL" />
+      </geometry>
+      <material
+        name="">
+        <color
+          rgba="0.792156862745098 0.819607843137255 0.933333333333333 1" />
+      </material>
+    </visual>
+    <collision>
+      <origin
+        xyz="0 0 0"
+        rpy="0 0 0" />
+      <geometry>
+        <mesh
+          filename="file://$(find piper_description)/meshes/link5.STL" />
       </geometry>
     </collision>
@@ -345,24 +291,15 @@
     name="link6">
     <inertial>
-      <origin
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
File: piper_description/urdf/piper_description_old.urdf (robot description, URDF)
Before this commit: robot piper, 10 links, 9 joints
Links:
- link link6: mass 0.007 -> 0.00699089613564366

File: piper_description/urdf/piper_no_gripper_description.urdf (robot description, URDF)
Before this commit: robot piper, 8 links, 7 joints
Links:
- removed link dummy_link
- link link6: mass 0.007 -> 0.00699089613564366
Joints:
- removed joint base_to_dummy
- joint joint6: limit lower=-2.0944 upper=2.0944 effort=100 velocity=3 -> lower=-2.0944 upper=2.0944 effort=100 velocity=5
